File: blinkenlights.kicad_pcb (KiCad board)
At the start: 2 copper layers, 80 x 80 mm, 61 parts, among them J101 ESP-01S, J102 PROG, J103 serial, J104 PWR, U101 AZ1117-3.3

Commit message: Konvert to KiCAD 6.x
KiCAD 6.x use a different file format and differetn file extentions
to store the data. Convert files to KiCAD 6.x.

Signed-off-by: Benedikt Spranger <b.spranger@linutronix.de>
Other:
- net class Default removed
